Commit message: new frame

File: sigma_cell.xacro (robot description, xacro)
@@ -6,5 +6,5 @@
 	<origin xyz= "0.63 0.40 0" rpy= "0 0 0"/>
 	<geometry>
-		<mesh filename="package://test/support/meshes/ur3e_frame.stl" scale='0.001 0.001 0.001'/>
+		<mesh filename="package://test/support/meshes/ur3e_frame_rack.stl" scale='0.001 0.001 0.001'/>
 	</geometry>
 	<material name="cell">
@@ -15,5 +15,5 @@
 	<origin xyz= "0.63 0.40 0" rpy= "0 0 0"/>
 	<geometry>
-		<mesh filename="package://test/support/meshes/ur3e_frame.stl" scale='0.001 0.001 0.001'/>
+		<mesh filename="package://test/support/meshes/ur3e_frame_rack.stl" scale='0.001 0.001 0.001'/>
 	</geometry>
 	</collision>
@@ -27,10 +27,10 @@
 <xacro:include filename="$(find ur_description)/urdf/ur3e.xacro"/>
 <joint name="base_joint" type="fixed">
-	<parent link="world" />
+	<parent link="cell_link" />
 	<child link = "base_link" />
 	<origin xyz="0 0 0.015" rpy="0 0 0"/>
 </joint>
 <xacro:include filename="$(find onrobot_2fg7_description)/urdf/onrobot_2fg7.xacro"/>
-<xacro:onrobot_2fg7_gripper  prefix="gripper_"/>
+<xacro:onrobot_2fg7_gripper  prefix="gripper_" finger_configuration="inwards"/>
 		<joint name="gripper_base_joint" type="fixed">
 		    <parent link="tool0" />

Commit message: Update program python

File: sigma_cell.xacro (robot description, xacro)
@@ -38,3 +38,9 @@
 		    <origin xyz="0 0 0" rpy="0 0 0"/>
 		</joint>
+<link name = "end_eff"> </link>
+<joint name = "gripper_end_eff" type = "fixed">
+	<parent  link="tool0"/>
+	<child link="end_eff"/>
+	<origin xyz = "0 0 0.1" rpy="0 0 0"/>
+	</joint>
 </robot>

Commit message: Marker Update

File: sigma_cell.xacro (robot description, xacro)
@@ -23,5 +23,5 @@
 	<parent link="world" />
 	<child link = "cell_link" />
-	<origin xyz= "0 0 0" rpy= "0 0 0"/>
+	<origin xyz= "0 0 0" rpy= "0 0 1.57"/>
 	</joint>
 <xacro:include filename="$(find ur_description)/urdf/ur3e.xacro"/>
