Commit message: Update xacro

File: sigma.xacro (robot description, xacro)
@@ -23,11 +23,11 @@
 	<parent link="world" />
 	<child link = "cell_link" />
-	<origin xyz= "0 0 0" rpy= "0 0 0"/>
+	<origin xyz= "0 0 0.05" rpy= "0 0 0"/>
 	</joint>
 <xacro:include filename="$(find ur_description)/urdf/ur3e.xacro"/>
 <joint name="base_joint" type="fixed">
-	<parent link="world" />
+	<parent link="cell_link" />
 	<child link = "base_link" />
-	<origin xyz="0 0 0.015" rpy="0 0 0"/>
+	<origin xyz="0 0 0.017" rpy="0 0 0"/>
 </joint>
 <link name = "end_eff"> </link>
