Commit message: Update of path V2

File: sigma_cell .xacro (robot description, xacro)
@@ -44,9 +44,3 @@
 		    <origin xyz="0 0 0" rpy="0 0 0"/>
 		</joint>
-<link name = "end_eff"> </link>
-<joint name = "gripper_end_eff" type = "fixed">
-	<parent  link="tool0"/>
-	<child link="end_eff"/>
-	<origin xyz = "0 0 0.1" rpy="0 0 0"/>
-	</joint>
 </robot>
